File: can_phys.kicad_sch (KiCad schematic)
At the start: 16 parts, among them J10 Hldx 120R, J11 Body 120R, U5 TJA1051T-3, U6 TJA1051T-3

Commit message: drawings: added title and project name
Other:
- company: (none) -> github.com/gabbla
- title: (none) -> CAN Phys
Changed lines of the file:
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@@
 	(generator_version "8.0")
 	(paper "A4")
+	(title_block
+		(title "CAN Phys")
+		(rev "v0.1.0")
+		(company "github.com/gabbla")
+		(comment 1 "${PROJECTNAME}")
+	)
 	(junction
 		(at 195.58 76.2)

Commit message: io, spi flash, stuff
Parts:
- renumbered C19 to C37, C20 to C38, C21 to C39, C22 to C40, C23 to C41, C24 to C42, J11 to J7, J10 to J8, R31 to R51, R32 to R52, R33 to R53, R34 to R54, U5 to U8, U6 to U9
Changed lines of the file:
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@@
 		(dnp no)
 		(fields_autoplaced yes)
-		(property "Reference" "C20"
+		(property "Reference" "C38"
 			(at 64.77 134.6135 0)
 			(effects
@@
 			(project "haldex_controller"
 				(path "/f9b060b2-b7a5-478e-9a0d-346ba4acb11f/96bb4d88-5f7d-436c-ad57-e0256ce9a962"
-					(reference "C20")
+					(reference "C38")
 					(unit 1)
 				)
@@
 		(dnp no)
 		(fields_autoplaced yes)
-		(property "Reference" "R33"
+		(property "Reference" "R53"
 			(at 198.12 124.4599 0)
 			(effects
@@
 			(project "haldex_controller"
 				(path "/f9b060b2-b7a5-478e-9a0d-346ba4acb11f/96bb4d88-5f7d-436c-ad57-e0256ce9a962"
-					(reference "R33")
+					(reference "R53")
 					(unit 1)
 				)
@@
 		(dnp no)
 		(fields_autoplaced yes)
-		(property "Reference" "C21"
+		(property "Reference" "C39"
 			(at 138.4363 46.99 90)
 			(effects
@@
 			(project "haldex_controller"
 				(path "/f9b060b2-b7a5-478e-9a0d-346ba4acb11f/96bb4d88-5f7d-436c-ad57-e0256ce9a962"
-					(reference "C21")
+					(reference "C39")
 					(unit 1)
 				)
@@
 		(dnp no)
 		(fields_autoplaced yes)
-		(property "Reference" "#PWR060"
+		(property "Reference" "#PWR0108"
 			(at 62.23 93.98 0)
 			(effects
@@
 			(project "haldex_controller"
 				(path "/f9b060b2-b7a5-478e-9a0d-346ba4acb11f/96bb4d88-5f7d-436c-ad57-e0256ce9a962"
-					(reference "#PWR060")
+					(reference "#PWR0108")
 					(unit 1)
 				)
@@
 		(dnp no)
 		(fields_autoplaced yes)
-		(property "Reference" "C24"
+		(property "Reference" "C42"
 			(at 208.2863 124.46 90)
 			(effects
@@
 			(project "haldex_controller"
 				(path "/f9b060b2-b7a5-478e-9a0d-346ba4acb11f/96bb4d88-5f7d-436c-ad57-e0256ce9a962"
-					(reference "C24")
+					(reference "C42")
 					(unit 1)
 				)
@@
 		(on_board yes)
 		(dnp no)
-		(property "Reference" "U6"
+		(property "Reference" "U9"
 			(at 118.872 113.284 0)
 			(effects
@@
 			(project "haldex_controller"
 				(path "/f9b060b2-b7a5-478e-9a0d-346ba4acb11f/96bb4d88-5f7d-436c-ad57-e0256ce9a962"
-					(reference "U6")
+					(reference "U9")
 					(unit 1)
 				)
@@
 		(dnp no)
 		(fields_autoplaced yes)
-		(property "Reference" "R31"
+		(property "Reference" "R51"
 			(at 198.12 69.8499 0)
 			(effects
@@
 			(project "haldex_controller"
 				(path "/f9b060b2-b7a5-478e-9a0d-346ba4acb11f/96bb4d88-5f7d-436c-ad57-e0256ce9a962"
-					(reference "R31")
+					(reference "R51")
 					(unit 1)
 				)
@@
 		(dnp no)
 		(fields_autoplaced yes)
-		(property "Reference" "R32"
+		(property "Reference" "R52"
 			(at 198.12 80.0099 0)
 			(effects
@@
 			(project "haldex_controller"
 				(path "/f9b060b2-b7a5-478e-9a0d-346ba4acb11f/96bb4d88-5f7d-436c-ad57-e0256ce9a962"
-					(reference "R32")
+					(reference "R52")
 					(unit 1)
 				)
@@
 		(dnp no)
 		(fields_autoplaced yes)
-		(property "Reference" "#PWR065"
+		(property "Reference" "#PWR0113"
 			(at 129.54 106.68 0)
 			(effects
@@
 			(project "haldex_controller"
 				(path "/f9b060b2-b7a5-478e-9a0d-346ba4acb11f/96bb4d88-5f7d-436c-ad57-e0256ce9a962"
-					(reference "#PWR065")
+					(reference "#PWR0113")
 					(unit 1)
 				)
@@
 		(dnp no)
 		(fields_autoplaced yes)
-		(property "Reference" "#PWR059"
+		(property "Reference" "#PWR0107"
 			(at 62.23 73.66 0)
 			(effects
@@
 			(project "haldex_controller"
 				(path "/f9b060b2-b7a5-478e-9a0d-346ba4acb11f/96bb4d88-5f7d-436c-ad57-e0256ce9a962"
-					(reference "#PWR059")
+					(reference "#PWR0107")
 					(unit 1)
 				)
@@
 		(dnp no)
 		(fields_autoplaced yes)
-		(property "Reference" "R34"
+		(property "Reference" "R54"
 			(at 198.12 134.6199 0)
 			(effects
@@
 			(project "haldex_controller"
 				(path "/f9b060b2-b7a5-478e-9a0d-346ba4acb11f/96bb4d88-5f7d-436c-ad57-e0256ce9a962"
-					(reference "R34")
+					(reference "R54")
 					(unit 1)
 				)
@@
 		(dnp no)
 		(fields_autoplaced yes)
-		(property "Reference" "#PWR068"
+		(property "Reference" "#PWR0116"
 			(at 149.86 116.84 0)
 			(effects
@@
 			(project "haldex_controller"
 				(path "/f9b060b2-b7a5-478e-9a0d-346ba4acb11f/96bb4d88-5f7d-436c-ad57-e0256ce9a962"
-					(reference "#PWR068")
+					(reference "#PWR0116")
 					(unit 1)
 				)
@@
 		(dnp no)
 		(fields_autoplaced yes)
-		(property "Reference" "#PWR063"
+		(property "Reference" "#PWR0111"
 			(at 129.54 52.07 0)
 			(effects
@@
 			(project "haldex_controller"
 				(path "/f9b060b2-b7a5-478e-9a0d-346ba4acb11f/96bb4d88-5f7d-436c-ad57-e0256ce9a962"
-					(reference "#PWR063")
+					(reference "#PWR0111")
 					(unit 1)
 				)
@@
 		(dnp no)
 		(fields_autoplaced yes)
-		(property "Reference" "#PWR070"
+		(property "Reference" "#PWR0118"
 			(at 213.36 139.7 0)
 			(effects
@@
 			(project "haldex_controller"
 				(path "/f9b060b2-b7a5-478e-9a0d-346ba4acb11f/96bb4d88-5f7d-436c-ad57-e0256ce9a962"
-					(reference "#PWR070")
+					(reference "#PWR0118")
 					(unit 1)
 				)
@@
 		(dnp no)
 		(fields_autoplaced yes)
-		(property "Reference" "#PWR064"
+		(property "Reference" "#PWR0112"
 			(at 129.54 91.44 0)
 			(effects
@@
 			(project "haldex_controller"
 				(path "/f9b060b2-b7a5-478e-9a0d-346ba4acb11f/96bb4d88-5f7d-436c-ad57-e0256ce9a962"
-					(reference "#PWR064")
+					(reference "#PWR0112")
 					(unit 1)
 				)
@@
 		(dnp no)
 		(fields_autoplaced yes)
-		(property "Reference" "#PWR067"
+		(property "Reference" "#PWR0115"
 			(at 149.86 62.23 0)
 			(effects
@@
 			(project "haldex_controller"
 				(path "/f9b060b2-b7a5-478e-9a0d-346ba4acb11f/96bb4d88-5f7d-436c-ad57-e0256ce9a962"
-					(reference "#PWR067")
+					(reference "#PWR0115")
 					(unit 1)
 				)
@@
 		(dnp no)
 		(fields_autoplaced yes)
-		(property "Reference" "#PWR061"
+		(property "Reference" "#PWR0109"
 			(at 62.23 128.27 0)
 			(effects
@@
 			(project "haldex_controller"
 				(path "/f9b060b2-b7a5-478e-9a0d-346ba4acb11f/96bb4d88-5f7d-436c-ad57-e0256ce9a962"
-					(reference "#PWR061")
+					(reference "#PWR0109")
 					(unit 1)
 				)
@@
 		(dnp no)
 		(fields_autoplaced yes)
-		(property "Reference" "J10"
+		(property "Reference" "J8"
 			(at 205.74 115.5699 0)
 			(effects
@@
 			(project "haldex_controller"
 				(path "/f9b060b2-b7a5-478e-9a0d-346ba4acb11f/96bb4d88-5f7d-436c-ad57-e0256ce9a962"
-					(reference "J10")
+					(reference "J8")
 					(unit 1)
 				)
@@
 		(on_board yes)
 		(dnp no)
-		(property "Reference" "U5"
+		(property "Reference" "U8"
 			(at 118.872 58.674 0)
 			(effects
@@
 			(project "haldex_controller"
 				(path "/f9b060b2-b7a5-478e-9a0d-346ba4acb11f/96bb4d88-5f7d-436c-ad57-e0256ce9a962"
-					(reference "U5")
+					(reference "U8")
 					(unit 1)
 				)
@@
 		(dnp no)
 		(fields_autoplaced yes)
-		(property "Reference" "#PWR062"
+		(property "Reference" "#PWR0110"
 			(at 62.23 148.59 0)
 			(effects
@@
 			(project "haldex_controller"
 				(path "/f9b060b2-b7a5-478e-9a0d-346ba4acb11f/96bb4d88-5f7d-436c-ad57-e0256ce9a962"
-					(reference "#PWR062")
+					(reference "#PWR0110")
 					(unit 1)
 				)
@@
 		(dnp no)
 		(fields_autoplaced yes)
-		(property "Reference" "#PWR069"
+		(property "Reference" "#PWR0117"
 			(at 213.36 85.09 0)
 			(effects
@@
 			(project "haldex_controller"
 				(path "/f9b060b2-b7a5-478e-9a0d-346ba4acb11f/96bb4d88-5f7d-436c-ad57-e0256ce9a962"
-					(reference "#PWR069")
+					(reference "#PWR0117")
 					(unit 1)
 				)
@@
 		(dnp no)
 		(fields_autoplaced yes)
-		(property "Reference" "#PWR066"
+		(property "Reference" "#PWR0114"
 			(at 129.54 146.05 0)
 			(effects
@@
 			(project "haldex_controller"
 				(path "/f9b060b2-b7a5-478e-9a0d-346ba4acb11f/96bb4d88-5f7d-436c-ad57-e0256ce9a962"
-					(reference "#PWR066")
+					(reference "#PWR0114")
 					(unit 1)
 				)
@@
 		(dnp no)
 		(fields_autoplaced yes)
-		(property "Reference" "C23"
+		(property "Reference" "C41"
 			(at 208.2863 69.85 90)
 			(effects
@@
 			(project "haldex_controller"
 				(path "/f9b060b2-b7a5-478e-9a0d-346ba4acb11f/96bb4d88-5f7d-436c-ad57-e0256ce9a962"
-					(reference "C23")
+					(reference "C41")
 					(unit 1)
 				)
@@
 		(dnp no)
 		(fields_autoplaced yes)
-		(property "Reference" "J11"
+		(property "Reference" "J7"
 			(at 205.74 60.9599 0)
 			(effects
@@
 			(project "haldex_controller"
 				(path "/f9b060b2-b7a5-478e-9a0d-346ba4acb11f/96bb4d88-5f7d-436c-ad57-e0256ce9a962"
-					(reference "J11")
+					(reference "J7")
 					(unit 1)
 				)
@@
 		(dnp no)
 		(fields_autoplaced yes)
-		(property "Reference" "C22"
+		(property "Reference" "C40"
 			(at 138.4363 101.6 90)
 			(effects
@@
 			(project "haldex_controller"
 				(path "/f9b060b2-b7a5-478e-9a0d-346ba4acb11f/96bb4d88-5f7d-436c-ad57-e0256ce9a962"
-					(reference "C22")
+					(reference "C40")
 					(unit 1)
 				)
@@
 		(dnp no)
 		(fields_autoplaced yes)
-		(property "Reference" "C19"
+		(property "Reference" "C37"
 			(at 64.77 80.0035 0)
 			(effects
@@
 			(project "haldex_controller"
 				(path "/f9b060b2-b7a5-478e-9a0d-346ba4acb11f/96bb4d88-5f7d-436c-ad57-e0256ce9a962"
-					(reference "C19")
-					(unit 1)
-				)
+					(reference "C37")
+					(unit 1)
+				)
