File: connectors.kicad_sch (KiCad schematic)
At the start: 12 parts, among them J12 Brake light, J13 Handbrake, J14 12V In, J6 Body, J7 Haldex, J8 K Line

Commit message: drawings: added title and project name
Other:
- company: (none) -> github.com/gabbla
- title: (none) -> Connectors
Changed lines of the file:
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@@
 	(generator_version "8.0")
 	(paper "A4")
+	(title_block
+		(title "Connectors")
+		(rev "v0.1.0")
+		(company "github.com/gabbla")
+		(comment 1 "${PROJECTNAME}")
+	)
 	(junction
 		(at 57.15 125.73)

Commit message: io, spi flash, stuff
Parts:
- removed D12, D13: PESD2CANFD27V-U, Package_TO_SOT_SMD:SOT-23, symbol Power_Protection:NUP2105L
- removed J6: Body, symbol Connector:Screw_Terminal_01x08
- removed J7: Haldex, symbol Connector:Screw_Terminal_01x08
- removed J8: K Line, Connector_PinHeader_2.54mm:PinHeader_1x02_P2.54mm_Horizontal, symbol Connector_Generic:Conn_01x02
- added D18, D19, D20: PESD2CANFD27V-U, Package_TO_SOT_SMD:SOT-23, symbol Power_Protection:NUP2105L
- added F3: 500mA, symbol Device:Fuse_Small
- added J11: K Line, Connector_PinHeader_2.54mm:PinHeader_1x02_P2.54mm_Horizontal, symbol Connector_Generic:Conn_01x02
- added J9: ECU Connector, symbol ecu_connector:ECU_CONN
- J12: value Brake light -> Brake Light
- renumbered J14 to J10
Connections:
- net +BATT: now also F3.1, J9.A1, J9.B1
- net BODY_BRAKE_LIGHT_SWITCH: now also J9.A2
- net BODY_CAN_H: now also D16.2 (K), J9.A7
- net BODY_CAN_L: now also D16.1 (K), J9.A6
- net BODY_HANDBRAKE: now also J9.A3
- net BODY_K_LINE: now also D15.1 (K), J11.1 (Pin_1), J9.A4; no longer D17.1 (K)
- net GNDPWR: now also D18.3 (A), D19.3 (A), D20.3 (A), J9.A8, J9.B8, J9.C8
- net HLDX_BRAKE_LIGHT_SWITCH: now also D17.1 (K), J9.B2; no longer D15.1 (K)
- net HLDX_CAN_H: now also D18.2 (K), J9.B7
- net HLDX_CAN_L: now also D18.1 (K), J9.B6
- net HLDX_HANDBRAKE: now also D17.2 (K), J9.B3; no longer D15.2 (K)
- net HLDX_K_LINE: now also D15.2 (K), J11.2 (Pin_2), J9.B4; no longer D16.1 (K)
- net VACANT: now also J9.A5, J9.B5
- new net USER_BATT: F3.2, J9.C1
- new net USER_INPUT_1: D19.1 (K), J9.C2
- new net USER_INPUT_2: D19.2 (K), J9.C3
- new net USER_OUTPUT_1: D20.1 (K), J9.C4
- new net USER_OUTPUT_2: D20.2 (K), J9.C5
Other:
- title: Connectors -> Connector
- moved on the sheet: J10
