File: connectors.kicad_sch (KiCad schematic)
At the start: 13 parts, among them J10 12V In, J11 K Line, J12 Brake Light, J13 Handbrake, J9 ECU Connector

Commit message: sch: fixing component footprints
Parts:
- F3: footprint (none) -> Fuse:Fuse_1206_3216Metric
- J10: value 12V In -> 12V in; footprint (none) -> TerminalBlock_Phoenix:TerminalBlock_Phoenix_MKDS-1,5-2-5.08_1x02_P5.08mm_Horizontal
- renumbered D14 to D15, D15 to D16, D16 to D17, D17 to D18, D18 to D19, D19 to D20, D20 to D21
Changed lines of the file:
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@@
 		(dnp no)
 		(fields_autoplaced yes)
-		(property "Reference" "D16"
+		(property "Reference" "D17"
 			(at 177.8 201.9299 0)
 			(effects
@@
 			(project "haldex_controller"
 				(path "/f9b060b2-b7a5-478e-9a0d-346ba4acb11f/439b2486-c84e-4eca-9430-b0865af9ee5e"
-					(reference "D16")
+					(reference "D17")
 					(unit 1)
 				)
@@
 		(dnp no)
 		(fields_autoplaced yes)
-		(property "Reference" "D15"
+		(property "Reference" "D16"
 			(at 146.05 201.9299 0)
 			(effects
@@
 			(project "haldex_controller"
 				(path "/f9b060b2-b7a5-478e-9a0d-346ba4acb11f/439b2486-c84e-4eca-9430-b0865af9ee5e"
-					(reference "D15")
+					(reference "D16")
 					(unit 1)
 				)
@@
 		(dnp no)
 		(fields_autoplaced yes)
-		(property "Reference" "#PWR0154"
+		(property "Reference" "#PWR0157"
 			(at 234.95 218.44 0)
 			(effects
@@
 			(project "haldex_controller"
 				(path "/f9b060b2-b7a5-478e-9a0d-346ba4acb11f/439b2486-c84e-4eca-9430-b0865af9ee5e"
-					(reference "#PWR0154")
+					(reference "#PWR0157")
 					(unit 1)
 				)
@@
 		(dnp no)
 		(fields_autoplaced yes)
-		(property "Reference" "D18"
+		(property "Reference" "D19"
 			(at 241.3 201.9299 0)
 			(effects
@@
 			(project "haldex_controller"
 				(path "/f9b060b2-b7a5-478e-9a0d-346ba4acb11f/439b2486-c84e-4eca-9430-b0865af9ee5e"
-					(reference "D18")
+					(reference "D19")
+					(unit 1)
+				)
+			)
+		)
+	)
+	(symbol
+		(lib_id "Connector:Screw_Terminal_01x02")
+		(at 106.68 43.18 180)
+		(unit 1)
+		(exclude_from_sim no)
+		(in_bom yes)
+		(on_board yes)
+		(dnp no)
+		(fields_autoplaced yes)
+		(property "Reference" "J10"
+			(at 106.68 34.29 0)
+			(effects
+				(font
+					(size 1.27 1.27)
+				)
+			)
+		)
+		(property "Value" "12V in"
+			(at 106.68 36.83 0)
+			(effects
+				(font
+					(size 1.27 1.27)
+				)
+			)
+		)
+		(property "Footprint" "TerminalBlock_Phoenix:TerminalBlock_Phoenix_MKDS-1,5-2-5.08_1x02_P5.08mm_Horizontal"
+			(at 106.68 43.18 0)
+			(effects
+				(font
+					(size 1.27 1.27)
+				)
+				(hide yes)
+			)
+		)
+		(property "Datasheet" "~"
+			(at 106.68 43.18 0)
+			(effects
+				(font
+					(size 1.27 1.27)
+				)
+				(hide yes)
+			)
+		)
+		(property "Description" "Generic screw terminal, single row, 01x02, script generated (kicad-library-utils/schlib/autogen/connector/)"
+			(at 106.68 43.18 0)
+			(effects
+				(font
+					(size 1.27 1.27)
+				)
+				(hide yes)
+			)
+		)
+		(pin "1"
+		)
+		(pin "2"
+		)
+		(instances
+			(project "haldex_controller"
+				(path "/f9b060b2-b7a5-478e-9a0d-346ba4acb11f/439b2486-c84e-4eca-9430-b0865af9ee5e"
+					(reference "J10")
 					(unit 1)
 				)
@@
 		(dnp no)
 		(fields_autoplaced yes)
-		(property "Reference" "#PWR0151"
+		(property "Reference" "#PWR0154"
 			(at 139.7 218.44 0)
 			(effects
@@
 			(project "haldex_controller"
 				(path "/f9b060b2-b7a5-478e-9a0d-346ba4acb11f/439b2486-c84e-4eca-9430-b0865af9ee5e"
-					(reference "#PWR0151")
+					(reference "#PWR0154")
 					(unit 1)
 				)
@@
 	)
 	(symbol
-		(lib_id "Connector:Screw_Terminal_01x02")
-		(at 106.68 43.18 180)
-		(unit 1)
-		(exclude_from_sim no)
-		(in_bom yes)
-		(on_board yes)
-		(dnp no)
-		(fields_autoplaced yes)
-		(property "Reference" "J10"
-			(at 106.68 34.29 0)
-			(effects
-				(font
-					(size 1.27 1.27)
-				)
-			)
-		)
-		(property "Value" "12V In"
-			(at 106.68 36.83 0)
-			(effects
-				(font
-					(size 1.27 1.27)
-				)
-			)
-		)
-		(property "Footprint" ""
-			(at 106.68 43.18 0)
-			(effects
-				(font
-					(size 1.27 1.27)
-				)
-				(hide yes)
-			)
-		)
-		(property "Datasheet" "~"
-			(at 106.68 43.18 0)
-			(effects
-				(font
-					(size 1.27 1.27)
-				)
-				(hide yes)
-			)
-		)
-		(property "Description" "Generic screw terminal, single row, 01x02, script generated (kicad-library-utils/schlib/autogen/connector/)"
-			(at 106.68 43.18 0)
-			(effects
-				(font
-					(size 1.27 1.27)
-				)
-				(hide yes)
-			)
-		)
-		(pin "1"
-		)
-		(pin "2"
-		)
-		(instances
-			(project "haldex_controller"
-				(path "/f9b060b2-b7a5-478e-9a0d-346ba4acb11f/439b2486-c84e-4eca-9430-b0865af9ee5e"
-					(reference "J10")
-					(unit 1)
-				)
-			)
-		)
-	)
-	(symbol
 		(lib_id "Power_Protection:NUP2105L")
 		(at 203.2 203.2 0)
@@
 		(dnp no)
 		(fields_autoplaced yes)
-		(property "Reference" "D17"
+		(property "Reference" "D18"
 			(at 209.55 201.9299 0)
 			(effects
@@
 			(project "haldex_controller"
 				(path "/f9b060b2-b7a5-478e-9a0d-346ba4acb11f/439b2486-c84e-4eca-9430-b0865af9ee5e"
-					(reference "D17")
+					(reference "D18")
 					(unit 1)
 				)
@@
 			)
 		)
-		(property "Footprint" ""
+		(property "Footprint" "Fuse:Fuse_1206_3216Metric"
 			(at 95.25 121.92 0)
 			(effects
@@
 		(dnp no)
 		(fields_autoplaced yes)
-		(property "Reference" "#PWR0150"
+		(property "Reference" "#PWR0153"
 			(at 118.11 54.61 0)
 			(effects
@@
 			(project "haldex_controller"
 				(path "/f9b060b2-b7a5-478e-9a0d-346ba4acb11f/439b2486-c84e-4eca-9430-b0865af9ee5e"
-					(reference "#PWR0150")
+					(reference "#PWR0153")
 					(unit 1)
 				)
@@
 		(dnp no)
 		(fields_autoplaced yes)
-		(property "Reference" "#PWR0153"
+		(property "Reference" "#PWR0156"
 			(at 203.2 218.44 0)
 			(effects
@@
 			(project "haldex_controller"
 				(path "/f9b060b2-b7a5-478e-9a0d-346ba4acb11f/439b2486-c84e-4eca-9430-b0865af9ee5e"
-					(reference "#PWR0153")
+					(reference "#PWR0156")
 					(unit 1)
 				)
@@
 		(dnp no)
 		(fields_autoplaced yes)
-		(property "Reference" "#PWR0155"
+		(property "Reference" "#PWR0158"
 			(at 266.7 218.44 0)
 			(effects
@@
 			(project "haldex_controller"
 				(path "/f9b060b2-b7a5-478e-9a0d-346ba4acb11f/439b2486-c84e-4eca-9430-b0865af9ee5e"
-					(reference "#PWR0155")
+					(reference "#PWR0158")
 					(unit 1)
 				)
@@
 		(dnp no)
 		(fields_autoplaced yes)
-		(property "Reference" "D19"
+		(property "Reference" "D20"
 			(at 273.05 201.9299 0)
 			(effects
@@
 			(project "haldex_controller"
 				(path "/f9b060b2-b7a5-478e-9a0d-346ba4acb11f/439b2486-c84e-4eca-9430-b0865af9ee5e"
-					(reference "D19")
+					(reference "D20")
 					(unit 1)
 				)
@@
 		(dnp no)
 		(fields_autoplaced yes)
-		(property "Reference" "#PWR0148"
+		(property "Reference" "#PWR0151"
 			(at 107.95 218.44 0)
 			(effects
@@
 			(project "haldex_controller"
 				(path "/f9b060b2-b7a5-478e-9a0d-346ba4acb11f/439b2486-c84e-4eca-9430-b0865af9ee5e"
-					(reference "#PWR0148")
+					(reference "#PWR0151")
 					(unit 1)
 				)
@@
 		(dnp no)
 		(fields_autoplaced yes)
-		(property "Reference" "#PWR0156"
+		(property "Reference" "#PWR0159"
 			(at 298.45 218.44 0)
 			(effects
@@
 			(project "haldex_controller"
 				(path "/f9b060b2-b7a5-478e-9a0d-346ba4acb11f/439b2486-c84e-4eca-9430-b0865af9ee5e"
-					(reference "#PWR0156")
+					(reference "#PWR0159")
 					(unit 1)
 				)
@@
 		(dnp no)
 		(fields_autoplaced yes)
-		(property "Reference" "#PWR0147"
+		(property "Reference" "#PWR0150"
 			(at 88.9 120.65 0)
 			(effects
@@
 			(project "haldex_controller"
 				(path "/f9b060b2-b7a5-478e-9a0d-346ba4acb11f/439b2486-c84e-4eca-9430-b0865af9ee5e"
-					(reference "#PWR0147")
+					(reference "#PWR0150")
 					(unit 1)
 				)
@@
 		(dnp no)
 		(fields_autoplaced yes)
-		(property "Reference" "#PWR0152"
+		(property "Reference" "#PWR0155"
 			(at 171.45 218.44 0)
 			(effects
@@
 			(project "haldex_controller"
 				(path "/f9b060b2-b7a5-478e-9a0d-346ba4acb11f/439b2486-c84e-4eca-9430-b0865af9ee5e"
-					(reference "#PWR0152")
+					(reference "#PWR0155")
 					(unit 1)
 				)
@@
 		(dnp no)
 		(fields_autoplaced yes)
-		(property "Reference" "#PWR0146"
+		(property "Reference" "#PWR0149"
 			(at 86.36 218.44 0)
 			(effects
@@
 			(project "haldex_controller"
 				(path "/f9b060b2-b7a5-478e-9a0d-346ba4acb11f/439b2486-c84e-4eca-9430-b0865af9ee5e"
-					(reference "#PWR0146")
+					(reference "#PWR0149")
 					(unit 1)
 				)
@@
 		(dnp no)
 		(fields_autoplaced yes)
-		(property "Reference" "#PWR0149"
+		(property "Reference" "#PWR0152"
 			(at 118.11 39.37 0)
 			(effects
@@
 			(project "haldex_controller"
 				(path "/f9b060b2-b7a5-478e-9a0d-346ba4acb11f/439b2486-c84e-4eca-9430-b0865af9ee5e"
-					(reference "#PWR0149")
+					(reference "#PWR0152")
 					(unit 1)
 				)
@@
 		(dnp no)
 		(fields_autoplaced yes)
-		(property "Reference" "D14"
+		(property "Reference" "D15"
 			(at 114.3 201.9299 0)
 			(effects
@@
 			(project "haldex_controller"
 				(path "/f9b060b2-b7a5-478e-9a0d-346ba4acb11f/439b2486-c84e-4eca-9430-b0865af9ee5e"
-					(reference "D14")
+					(reference "D15")
 					(unit 1)
 				)
@@
 		(dnp no)
 		(fields_autoplaced yes)
-		(property "Reference" "D20"
+		(property "Reference" "D21"
 			(at 304.8 201.9299 0)
 			(effects
@@
 			(project "haldex_controller"
 				(path "/f9b060b2-b7a5-478e-9a0d-346ba4acb11f/439b2486-c84e-4eca-9430-b0865af9ee5e"
-					(reference "D20")
-					(unit 1)
-				)
+					(reference "D21")
+					(unit 1)
+				)

Commit message: sch: added footprint association
Parts:
- J9: footprint (none) -> ecu24:ecu24
Changed lines of the file:
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@@
 			)
 		)
-		(property "Footprint" ""
+		(property "Footprint" "ecu24:ecu24"
 			(at 81.28 118.11 0)
 			(effects

Commit message: sch: J10 footprint update
Parts:
- J10: footprint TerminalBlock_Phoenix:TerminalBlock_Phoenix_MKDS-1,5-2-5.08_1x02_P5.08mm_Horizontal -> TerminalBlock_Phoenix:TerminalBlock_Phoenix_PT-1,5-2-3.5-H_1x02_P3.50mm_Horizontal
Changed lines of the file:
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@@
 			)
 		)
-		(property "Footprint" "TerminalBlock_Phoenix:TerminalBlock_Phoenix_MKDS-1,5-2-5.08_1x02_P5.08mm_Horizontal"
+		(property "Footprint" "TerminalBlock_Phoenix:TerminalBlock_Phoenix_PT-1,5-2-3.5-H_1x02_P3.50mm_Horizontal"
 			(at 106.68 43.18 0)
 			(effects

Commit message: brd: routing in progress
Connections:
- net USER_INPUT_1: now also D20.2 (K); no longer D20.1 (K)
- net USER_INPUT_2: now also D20.1 (K); no longer D20.2 (K)
- net USER_OUTPUT_1: now also D21.2 (K); no longer D21.1 (K)
- net USER_OUTPUT_2: now also D21.1 (K); no longer D21.2 (K)
Changed lines of the file:
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@@
-	)
-	(junction
-		(at 269.24 172.72)
-		(diameter 0)
-		(color 0 0 0 0)
 	)
 	(junction
@@
 	)
 	(junction
-		(at 295.91 175.26)
-		(diameter 0)
-		(color 0 0 0 0)
-	)
-	(junction
-		(at 300.99 177.8)
-		(diameter 0)
-		(color 0 0 0 0)
-	)
-	(junction
 		(at 88.9 121.92)
 		(diameter 0)
@@
 	)
 	(junction
+		(at 300.99 175.26)
+		(diameter 0)
+		(color 0 0 0 0)
+	)
+	(junction
 		(at 185.42 147.32)
 		(diameter 0)
@@
 	)
 	(junction
+		(at 264.16 172.72)
+		(diameter 0)
+		(color 0 0 0 0)
+	)
+	(junction
 		(at 151.13 129.54)
 		(diameter 0)
@@
 	)
 	(junction
+		(at 295.91 177.8)
+		(diameter 0)
+		(color 0 0 0 0)
+	)
+	(junction
 		(at 182.88 124.46)
 		(diameter 0)
@@
 	)
 	(junction
+		(at 269.24 170.18)
+		(diameter 0)
+		(color 0 0 0 0)
+	)
+	(junction
 		(at 173.99 137.16)
 		(diameter 0)
@@
 	(junction
 		(at 105.41 124.46)
-		(diameter 0)
-		(color 0 0 0 0)
-	)
-	(junction
-		(at 264.16 170.18)
 		(diameter 0)
 		(color 0 0 0 0)
@@
 	(wire
 		(pts
-			(xy 300.99 177.8) (xy 300.99 198.12)
+			(xy 269.24 170.18) (xy 334.01 170.18)
 		)
 		(stroke
@@
 	(wire
 		(pts
+			(xy 264.16 172.72) (xy 334.01 172.72)
+		)
+		(stroke
+			(width 0)
+			(type default)
+		)
+	)
+	(wire
+		(pts
 			(xy 83.82 124.46) (xy 105.41 124.46)
 		)
@@
 	(wire
 		(pts
+			(xy 264.16 172.72) (xy 264.16 198.12)
+		)
+		(stroke
+			(width 0)
+			(type default)
+		)
+	)
+	(wire
+		(pts
 			(xy 83.82 139.7) (xy 86.36 139.7)
 		)
@@
 	(wire
 		(pts
+			(xy 295.91 177.8) (xy 295.91 198.12)
+		)
+		(stroke
+			(width 0)
+			(type default)
+		)
+	)
+	(wire
+		(pts
 			(xy 86.36 139.7) (xy 86.36 162.56)
 		)
@@
 	(wire
 		(pts
+			(xy 300.99 175.26) (xy 334.01 175.26)
+		)
+		(stroke
+			(width 0)
+			(type default)
+		)
+	)
+	(wire
+		(pts
 			(xy 153.67 114.3) (xy 153.67 152.4)
 		)
@@
 	(wire
 		(pts
-			(xy 264.16 170.18) (xy 334.01 170.18)
-		)
-		(stroke
-			(width 0)
-			(type default)
-		)
-	)
-	(wire
-		(pts
 			(xy 83.82 167.64) (xy 101.6 167.64)
 		)
@@
 	(wire
 		(pts
-			(xy 295.91 175.26) (xy 295.91 198.12)
+			(xy 269.24 170.18) (xy 269.24 198.12)
 		)
 		(stroke
@@
 	(wire
 		(pts
-			(xy 269.24 172.72) (xy 334.01 172.72)
-		)
-		(stroke
-			(width 0)
-			(type default)
-		)
-	)
-	(wire
-		(pts
 			(xy 86.36 162.56) (xy 86.36 185.42)
 		)
@@
 	(wire
 		(pts
-			(xy 83.82 170.18) (xy 264.16 170.18)
-		)
-		(stroke
-			(width 0)
-			(type default)
-		)
-	)
-	(wire
-		(pts
-			(xy 264.16 170.18) (xy 264.16 198.12)
+			(xy 83.82 170.18) (xy 269.24 170.18)
 		)
 		(stroke
@@
 	(wire
 		(pts
-			(xy 300.99 177.8) (xy 334.01 177.8)
-		)
-		(stroke
-			(width 0)
-			(type default)
-		)
-	)
-	(wire
-		(pts
 			(xy 232.41 157.48) (xy 232.41 198.12)
 		)
@@
 	(wire
 		(pts
-			(xy 83.82 172.72) (xy 269.24 172.72)
+			(xy 300.99 175.26) (xy 300.99 198.12)
+		)
+		(stroke
+			(width 0)
+			(type default)
+		)
+	)
+	(wire
+		(pts
+			(xy 83.82 172.72) (xy 264.16 172.72)
 		)
 		(stroke
@@
 	(wire
 		(pts
-			(xy 83.82 177.8) (xy 300.99 177.8)
+			(xy 83.82 177.8) (xy 295.91 177.8)
 		)
 		(stroke
@@
 	(wire
 		(pts
-			(xy 269.24 172.72) (xy 269.24 198.12)
-		)
-		(stroke
-			(width 0)
-			(type default)
-		)
-	)
-	(wire
-		(pts
 			(xy 83.82 157.48) (xy 232.41 157.48)
 		)
@@
 	(wire
 		(pts
-			(xy 83.82 175.26) (xy 295.91 175.26)
+			(xy 83.82 175.26) (xy 300.99 175.26)
 		)
 		(stroke
@@
 	(wire
 		(pts
-			(xy 295.91 175.26) (xy 334.01 175.26)
-		)
-		(stroke
+			(xy 295.91 177.8) (xy 334.01 177.8)
+		)
+		(stroke

Commit message: brd: layout complete
Parts:
- removed J11: K Line, Connector_PinHeader_2.54mm:PinHeader_1x02_P2.54mm_Horizontal, symbol Connector_Generic:Conn_01x02
- removed J12: Brake Light, Connector_PinHeader_2.54mm:PinHeader_1x02_P2.54mm_Horizontal, symbol Connector_Generic:Conn_01x02
- removed J13: Handbrake, Connector_PinHeader_2.54mm:PinHeader_1x02_P2.54mm_Horizontal, symbol Connector_Generic:Conn_01x02
- added JP1: K Line, Jumper:SolderJumper-2_P1.3mm_Open_TrianglePad1.0x1.5mm, symbol Jumper:SolderJumper_2_Open
- added JP2: Brake Light, Jumper:SolderJumper-2_P1.3mm_Open_TrianglePad1.0x1.5mm, symbol Jumper:SolderJumper_2_Open
- added JP3: Handbrake, Jumper:SolderJumper-2_P1.3mm_Open_TrianglePad1.0x1.5mm, symbol Jumper:SolderJumper_2_Open
Connections:
- net BODY_BRAKE_LIGHT_SWITCH: now also JP2.1 (A)
- net BODY_HANDBRAKE: now also JP3.1 (A)
- net BODY_K_LINE: now also JP1.1 (A)
- net HLDX_BRAKE_LIGHT_SWITCH: now also JP2.2 (B)
- net HLDX_HANDBRAKE: now also JP3.2 (B)
- net HLDX_K_LINE: now also JP1.2 (B)
