File: haldex_controller.kicad_sch (KiCad schematic)
At the start: 2 parts

Commit message: drawings: added title and project name
Other:
- company: (none) -> github.com/gabbla
Changed lines of the file:
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@@
 	(generator_version "8.0")
 	(paper "A3")
+	(title_block
+		(rev "v0.1.0")
+		(company "github.com/gabbla")
+		(comment 1 "${PROJECTNAME}")
+	)
 	(no_connect
 		(at 201.93 160.02)

Commit message: io, spi flash, stuff
Parts:
- renumbered R48 to R1, R49 to R2
Other:
- sheet Connectors renamed Connector
- sheet Vehicle signals renamed Signals
- added sheet Stackup (stackup.kicad_sch)
- sheet Connector ports: added USER_INPUT_1, USER_INPUT_2, USER_OUTPUT_1, USER_OUTPUT_2; removed none
- sheet MCU ports: added MCU_USER_INPUT_1, MCU_USER_INPUT_2, MCU_USER_OUTPUT_1, MCU_USER_OUTPUT_2; removed none
- sheet Signals ports: added MCU_USER_INPUT_1, MCU_USER_INPUT_2, MCU_USER_OUTPUT_1, MCU_USER_OUTPUT_2, USER_INPUT_1, USER_INPUT_2, USER_OUTPUT_1, USER_OUTPUT_2; removed none
