File: haldex_controller.kicad_sch (KiCad schematic)
At the start: 2 parts

Commit message: brd: layout complete
Parts:
- added J15: nRF7002 Ext, Connector_PinHeader_1.27mm:PinHeader_2x05_P1.27mm_Vertical, symbol Connector_Generic:Conn_02x05_Odd_Even
Connections:
- net MCU/SPI1_MISO: now also J15.7 (Pin_7)
- net MCU/SPI1_MOSI: now also J15.5 (Pin_5)
- net MCU/SPI1_SCK: now also J15.9 (Pin_9)
- net MCU/SPI1_~{CS}: now also J15.3 (Pin_3)
- net MCU/nRF7002_BUCK_EN: now also J15.2 (Pin_2)
- net MCU/nRF7002_IRQ: now also J15.1 (Pin_1)
- net MCU/nRF7002_VDDIO_EN: now also J15.4 (Pin_4)
- new net +3V3: J15.6 (Pin_6)
- new net GND: J15.10 (Pin_10), J15.8 (Pin_8)
- no-connect marks 2 -> 0
Other:
- removed sheet WiFi nRF7002
