File: power.kicad_sch (KiCad schematic)
At the start: 51 parts, among them IC4 TPS62A02DRLR, J9 GND, Q1 STR1550, Q2 BC807, Q3 PMOS, U3 LMR33630BDDA

Commit message: drawings: added title and project name
Other:
- company: (none) -> github.com/gabbla
- title: (none) -> Power
Changed lines of the file:
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@@
 	(generator_version "8.0")
 	(paper "A3")
+	(title_block
+		(title "Power")
+		(rev "v0.1.0")
+		(company "github.com/gabbla")
+		(comment 1 "${PROJECTNAME}")
+	)
 	(junction
 		(at 166.37 212.09)

Commit message: io, spi flash, stuff
Parts:
- renumbered C4 to C1, C40 to C10, C5 to C2, C6 to C3, C7 to C4, C8 to C5, C9 to C6, C10 to C7, C38 to C8, C39 to C9, D2 to D1, D3 to D2, D4 to D3, D18 to D4, FB6 to FB3, FB7 to FB4, H3 to H2, H2 to H3, IC4 to IC1, J9 to J1, L6 to L4, R13 to R10, R50 to R11, R51 to R12, R52 to R13, R53 to R14, R2 to R3, R3 to R4, R8 to R5, R9 to R6, R10 to R7, R11 to R8, R12 to R9, TP10 to TP1, TP3 to TP2, TP7 to TP3, TP9 to TP4, TP8 to TP5, U3 to U1
