File: usb.kicad_sch (KiCad schematic)
At the start: 7 parts, among them J2 USB, U4 USBLC6-2SC6

Commit message: drawings: added title and project name
Other:
- company: (none) -> github.com/gabbla
- title: (none) -> USB-C
Changed lines of the file:
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@@
 	(generator_version "8.0")
 	(paper "A4")
+	(title_block
+		(title "USB-C")
+		(rev "v0.1.0")
+		(company "github.com/gabbla")
+		(comment 1 "${PROJECTNAME}")
+	)
 	(junction
 		(at 138.43 81.28)

Commit message: io, spi flash, stuff
Parts:
- renumbered FB3 to FB5, J2 to J5, R6 to R38, R7 to R39, U4 to U6
Changed lines of the file:
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@@
 		(dnp no)
 		(fields_autoplaced yes)
-		(property "Reference" "#PWR032"
+		(property "Reference" "#PWR074"
 			(at 138.43 113.03 0)
 			(effects
@@
 			(project "haldex_controller"
 				(path "/f9b060b2-b7a5-478e-9a0d-346ba4acb11f/043ef3bc-15f0-4a00-a1c6-c31e1a8ee615"
-					(reference "#PWR032")
+					(reference "#PWR074")
 					(unit 1)
 				)
@@
 		(dnp no)
 		(fields_autoplaced yes)
-		(property "Reference" "#FLG011"
+		(property "Reference" "#FLG09"
 			(at 167.005 81.28 0)
 			(effects
@@
 			(project "haldex_controller"
 				(path "/f9b060b2-b7a5-478e-9a0d-346ba4acb11f/043ef3bc-15f0-4a00-a1c6-c31e1a8ee615"
-					(reference "#FLG011")
+					(reference "#FLG09")
 					(unit 1)
 				)
@@
 		(on_board yes)
 		(dnp no)
-		(property "Reference" "FB3"
+		(property "Reference" "FB5"
 			(at 148.59 75.184 90)
 			(effects
@@
 			(project "haldex_controller"
 				(path "/f9b060b2-b7a5-478e-9a0d-346ba4acb11f/043ef3bc-15f0-4a00-a1c6-c31e1a8ee615"
-					(reference "FB3")
+					(reference "FB5")
 					(unit 1)
 				)
@@
 		(dnp no)
 		(fields_autoplaced yes)
-		(property "Reference" "#PWR034"
+		(property "Reference" "#PWR076"
 			(at 209.55 90.17 0)
 			(effects
@@
 			(project "haldex_controller"
 				(path "/f9b060b2-b7a5-478e-9a0d-346ba4acb11f/043ef3bc-15f0-4a00-a1c6-c31e1a8ee615"
-					(reference "#PWR034")
+					(reference "#PWR076")
 					(unit 1)
 				)
@@
 		(dnp no)
 		(fields_autoplaced yes)
-		(property "Reference" "#PWR033"
+		(property "Reference" "#PWR075"
 			(at 160.02 80.01 0)
 			(effects
@@
 			(project "haldex_controller"
 				(path "/f9b060b2-b7a5-478e-9a0d-346ba4acb11f/043ef3bc-15f0-4a00-a1c6-c31e1a8ee615"
-					(reference "#PWR033")
+					(reference "#PWR075")
 					(unit 1)
 				)
@@
 		(on_board yes)
 		(dnp no)
-		(property "Reference" "U4"
+		(property "Reference" "U6"
 			(at 140.208 88.9 0)
 			(effects
@@
 			(project "haldex_controller"
 				(path "/f9b060b2-b7a5-478e-9a0d-346ba4acb11f/043ef3bc-15f0-4a00-a1c6-c31e1a8ee615"
-					(reference "U4")
+					(reference "U6")
 					(unit 1)
 				)
@@
 		(on_board yes)
 		(dnp no)
-		(property "Reference" "R7"
+		(property "Reference" "R39"
 			(at 203.2 75.946 90)
 			(effects
@@
 			(project "haldex_controller"
 				(path "/f9b060b2-b7a5-478e-9a0d-346ba4acb11f/043ef3bc-15f0-4a00-a1c6-c31e1a8ee615"
-					(reference "R7")
+					(reference "R39")
 					(unit 1)
 				)
@@
 		(dnp no)
 		(fields_autoplaced yes)
-		(property "Reference" "#PWR030"
+		(property "Reference" "#PWR072"
 			(at 93.98 128.27 0)
 			(effects
@@
 			(project "haldex_controller"
 				(path "/f9b060b2-b7a5-478e-9a0d-346ba4acb11f/043ef3bc-15f0-4a00-a1c6-c31e1a8ee615"
-					(reference "#PWR030")
+					(reference "#PWR072")
 					(unit 1)
 				)
@@
 		(on_board yes)
 		(dnp no)
-		(property "Reference" "J2"
+		(property "Reference" "J5"
 			(at 101.6 74.422 0)
 			(effects
@@
 			(project "haldex_controller"
 				(path "/f9b060b2-b7a5-478e-9a0d-346ba4acb11f/043ef3bc-15f0-4a00-a1c6-c31e1a8ee615"
-					(reference "J2")
+					(reference "J5")
 					(unit 1)
 				)
@@
 		(dnp no)
 		(fields_autoplaced yes)
-		(property "Reference" "#PWR031"
+		(property "Reference" "#PWR073"
 			(at 101.6 128.27 0)
 			(effects
@@
 			(project "haldex_controller"
 				(path "/f9b060b2-b7a5-478e-9a0d-346ba4acb11f/043ef3bc-15f0-4a00-a1c6-c31e1a8ee615"
-					(reference "#PWR031")
+					(reference "#PWR073")
 					(unit 1)
 				)
@@
 		(on_board yes)
 		(dnp no)
-		(property "Reference" "R6"
+		(property "Reference" "R38"
 			(at 203.2 68.326 90)
 			(effects
@@
 			(project "haldex_controller"
 				(path "/f9b060b2-b7a5-478e-9a0d-346ba4acb11f/043ef3bc-15f0-4a00-a1c6-c31e1a8ee615"
-					(reference "R6")
-					(unit 1)
-				)
+					(reference "R38")
+					(unit 1)
+				)
