File: vehicle_signals.kicad_sch (KiCad schematic)
At the start: 16 parts, among them IC3 TLIN1027DRQ1, U2 LTV-827S, U8 LTV-827S

Commit message: drawings: added title and project name
Other:
- company: (none) -> github.com/gabbla
- title: (none) -> Vehicle Signals
Changed lines of the file:
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@@
 	(generator_version "8.0")
 	(paper "A4")
+	(title_block
+		(title "Vehicle Signals")
+		(rev "v0.1.0")
+		(company "github.com/gabbla")
+		(comment 1 "${PROJECTNAME}")
+	)
 	(junction
 		(at 80.01 160.02)

Commit message: io, spi flash, stuff
Parts:
- added R57, R58, R65, R66: R_Small, Resistor_SMD:R_0603_1608Metric_Pad0.98x0.95mm_HandSolder, symbol Device:R_Small
- added R61, R62: 10k, Resistor_SMD:R_0603_1608Metric_Pad0.98x0.95mm_HandSolder, symbol Device:R_Small
- added U11, U13: LTV-827S, Package_DIP:SMDIP-8_W9.53mm, symbol Isolator:LTV-827S
- renumbered C41 to C43, C42 to C44, D19 to D13, IC3 to IC4, R47 to R55, R54 to R56, R57 to R59, R58 to R60, R45 to R63, R46 to R64, R55 to R67, R56 to R68, R44 to R69, R59 to R70, U8 to U10, U2 to U12
Connections:
- net +3V3: now also R61.2, R62.2
- net GND: now also U11.5, U11.7, U13.2, U13.4
- new net: R66.2, U13.3
- new net: R65.2, U13.1
- new net: R57.2, U11.1
- new net: R58.2, U11.3
- new net GNDPWR: U11.2, U11.4, U13.5, U13.7
- new net MCU_USER_INPUT_1: R61.1, U11.8
- new net MCU_USER_INPUT_2: R62.1, U11.6
- new net MCU_USER_OUTPUT_1: R65.1
- new net MCU_USER_OUTPUT_2: R66.1
- new net USER_INPUT_1: R57.1
- new net USER_INPUT_2: R58.1
- new net USER_OUTPUT_1: U13.8
- new net USER_OUTPUT_2: U13.6
Other:
- note added: "From MCU to user"
- note added: "From user to MCU"
- note added: "User output open-drain max 50mA Any protection?"
- moved on the sheet: C43, C44, D13, IC4, R55, R56, R59, R60, R63, R64, R67, R68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
