File: wifi_bt.kicad_sch (KiCad schematic)
At the start: 29 parts, among them IC1 LBEE5KL1YN-814, J3 Conn_Coaxial_Small, X2 32.768kHz

Commit message: drawings: added title and project name
Other:
- company: (none) -> github.com/gabbla
- title: (none) -> WiFi and Bluetooth - Murata 1YN
Changed lines of the file:
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@@
 	(generator_version "8.0")
 	(paper "A4")
+	(title_block
+		(title "WiFi and Bluetooth - Murata 1YN")
+		(rev "v0.1.0")
+		(company "github.com/gabbla")
+		(comment 1 "${PROJECTNAME}")
+	)
 	(junction
 		(at 151.13 57.15)

Commit message: io, spi flash, stuff
Parts:
- renumbered C16 to C31, C15 to C32, C13 to C33, C17 to C34, C14 to C35, C18 to C36, FB4 to FB7, IC1 to IC3, J3 to J6, L4 to L6, R18 to R42, R19 to R43, R14 to R44, R15 to R45, R16 to R46, R17 to R47, R20 to R48, R21 to R49, R22 to R50, TP14 to TP10, TP15 to TP11, TP16 to TP12, TP4 to TP13, TP11 to TP14, TP12 to TP15, TP13 to TP16, X2 to X1
