File: wifi_bt.kicad_sch (KiCad schematic)
At the start: 29 parts, among them IC3 LBEE5KL1YN-814, J6 Conn_Coaxial_Small, X1 32.768kHz

Commit message: sch: fixing component footprints
Parts:
- removed AE1: W3000, symbol Device:Antenna
- added ANT1: W3000, W3000:W3000, symbol W3000:W3000
- FB7, FB8: footprint (none) -> Inductor_SMD:L_0805_2012Metric_Pad1.05x1.20mm_HandSolder
- IC3: footprint LBEE5KL1YN814 -> LBEE5KL1YN-814:LBEE5KL1YN814
- J6: footprint (none) -> Connector_Coaxial:SMA_Amphenol_132134-10_Vertical
- L6: value 2u2 -> LQM18PN2R2MGH; footprint (none) -> Inductor_SMD:L_0603_1608Metric_Pad1.05x0.95mm_HandSolder
Connections:
- net at R50.1: now also ANT1.1 (FEED)
- no-connect marks 5 -> 6
Other:
- note removed: "LQM18PN2R2MGH"
- moved on the sheet: C34, C36, J6, R47, R48, R49, R50

Commit message: sch: fix footprint association for J6
Parts:
- J6: footprint Connector_Coaxial:SMA_Amphenol_132134-10_Vertical -> Connector_Coaxial:U.FL_Molex_MCRF_73412-0110_Vertical
Changed lines of the file:
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@@
 			)
 		)
-		(property "Footprint" "Connector_Coaxial:SMA_Amphenol_132134-10_Vertical"
+		(property "Footprint" "Connector_Coaxial:U.FL_Molex_MCRF_73412-0110_Vertical"
 			(at 198.12 119.38 0)
 			(effects

Commit message: brd: routing in progress
Parts:
- removed ANT1: W3000, W3000:W3000, symbol W3000:W3000
- removed FB8: FerriteBead_Small, Inductor_SMD:L_0805_2012Metric_Pad1.05x1.20mm_HandSolder, symbol Device:FerriteBead_Small
- removed J6: Conn_Coaxial_Small, Connector_Coaxial:U.FL_Molex_MCRF_73412-0110_Vertical, symbol Connector:Conn_Coaxial_Small
- removed R48, R50: 0, Resistor_SMD:R_0402_1005Metric_Pad0.72x0.64mm_HandSolder, symbol Device:R_Small
- removed TP10: SDIO_CMD, TestPoint:TestPoint_Pad_D1.0mm, symbol Connector:TestPoint
- removed TP11: SDIO_DATA_2, TestPoint:TestPoint_Pad_D1.0mm, symbol Connector:TestPoint
- removed TP12: SDIO_CLK, TestPoint:TestPoint_Pad_D1.0mm, symbol Connector:TestPoint
- removed TP14: SDIO_DATA_0, TestPoint:TestPoint_Pad_D1.0mm, symbol Connector:TestPoint
- removed TP15: SDIO_DATA_3, TestPoint:TestPoint_Pad_D1.0mm, symbol Connector:TestPoint
- removed TP16: SDIO_DATA_1, TestPoint:TestPoint_Pad_D1.0mm, symbol Connector:TestPoint
- added AE1: type1YN-antenna-p2ml4452-1, 1yn_antenna:1YN_ANTENNA, symbol Device:Antenna
- added C48, C49: 4p7, Capacitor_SMD:C_0402_1005Metric_Pad0.74x0.62mm_HandSolder, symbol Device:C_Small
- added J6: MM8130-2600RA2, MM8130-2600RA2:MM81302600RA2, symbol MM8130-2600RA2:MM8130-2600RA2
- added L9: LQW15AN2N4B00D, Inductor_SMD:L_0402_1005Metric, symbol Device:L_Small
- R42, R43, R44, R45, R46: footprint Resistor_SMD:R_0603_1608Metric_Pad0.98x0.95mm_HandSolder -> Resistor_SMD:R_0402_1005Metric_Pad0.72x0.64mm_HandSolder
- R47: now fitted
Connections:
- net SR_PVSS is gone; now on net GND: C33.2, C35.2, IC3.32 (GND_(SR_PVSS)_1), IC3.33 (GND_(SR_PVSS)_2)
- net ANT_FEED: now also J6.1 (IN); no longer R47.1
- net GND: now also C48.1, C49.1, J6.3 (GND), J6.4 (GND), J6.5 (GND), J6.6 (GND)
- net at C36.2, R49.1: now also R47.2, C48.2
- net at C34.2, R49.2: now also J6.2 (OUT)
- new net: C49.2, L9.1, R47.1
- new net: AE1.1 (A), L9.2
- no-connect marks 6 -> 5
Other:
- note removed: "GND(SR_PVSS) have to be isolated from typical GND"
- moved on the sheet: C34, C36, R49
