File: wifi_nrf7002.kicad_sch (KiCad schematic)
At the start: 13 parts, among them IC2 TPS2553DBVT

Commit message: drawings: added title and project name
Other:
- company: (none) -> github.com/gabbla
- title: (none) -> WiFi - Nordic nRF7002
Changed lines of the file:
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@@
 	(generator_version "8.0")
 	(paper "A4")
+	(title_block
+		(title "WiFi - Nordic nRF7002")
+		(rev "v0.1.0")
+		(company "github.com/gabbla")
+		(comment 1 "${PROJECTNAME}")
+	)
 	(junction
 		(at 132.08 95.25)

Commit message: io, spi flash, stuff
Parts:
- renumbered C37 to C27, C36 to C28, C25 to C29, C26 to C30, FB5 to FB6, R43 to R40, R42 to R41, TP5 to TP6, TP6 to TP7, TP1 to TP8, TP2 to TP9
Changed lines of the file:
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@@
 		(dnp no)
 		(fields_autoplaced yes)
-		(property "Reference" "TP1"
+		(property "Reference" "TP8"
 			(at 136.398 105.41 90)
 			(effects
@@
 			(project "haldex_controller"
 				(path "/f9b060b2-b7a5-478e-9a0d-346ba4acb11f/ac628dfb-9786-4488-a934-d1527b457eba"
-					(reference "TP1")
+					(reference "TP8")
 					(unit 1)
 				)
@@
 		(dnp no)
 		(fields_autoplaced yes)
-		(property "Reference" "C25"
+		(property "Reference" "C29"
 			(at 146.05 74.9362 0)
 			(effects
@@
 			(project "haldex_controller"
 				(path "/f9b060b2-b7a5-478e-9a0d-346ba4acb11f/ac628dfb-9786-4488-a934-d1527b457eba"
-					(reference "C25")
+					(reference "C29")
 					(unit 1)
 				)
@@
 		(dnp no)
 		(fields_autoplaced yes)
-		(property "Reference" "#PWR072"
+		(property "Reference" "#PWR082"
 			(at 143.51 87.63 0)
 			(effects
@@
 			(project "haldex_controller"
 				(path "/f9b060b2-b7a5-478e-9a0d-346ba4acb11f/ac628dfb-9786-4488-a934-d1527b457eba"
-					(reference "#PWR072")
+					(reference "#PWR082")
 					(unit 1)
 				)
@@
 		(dnp no)
 		(fields_autoplaced yes)
-		(property "Reference" "#PWR071"
+		(property "Reference" "#PWR077"
 			(at 36.83 68.58 0)
 			(effects
@@
 			(project "haldex_controller"
 				(path "/f9b060b2-b7a5-478e-9a0d-346ba4acb11f/ac628dfb-9786-4488-a934-d1527b457eba"
-					(reference "#PWR071")
+					(reference "#PWR077")
 					(unit 1)
 				)
@@
 		(dnp no)
 		(fields_autoplaced yes)
-		(property "Reference" "TP5"
+		(property "Reference" "TP6"
 			(at 76.708 107.95 90)
 			(effects
@@
 			(project "haldex_controller"
 				(path "/f9b060b2-b7a5-478e-9a0d-346ba4acb11f/ac628dfb-9786-4488-a934-d1527b457eba"
-					(reference "TP5")
+					(reference "TP6")
 					(unit 1)
 				)
@@
 		(dnp no)
 		(fields_autoplaced yes)
-		(property "Reference" "R42"
+		(property "Reference" "R41"
 			(at 105.41 102.8699 0)
 			(effects
@@
 			(project "haldex_controller"
 				(path "/f9b060b2-b7a5-478e-9a0d-346ba4acb11f/ac628dfb-9786-4488-a934-d1527b457eba"
-					(reference "R42")
+					(reference "R41")
 					(unit 1)
 				)
@@
 		(dnp no)
 		(fields_autoplaced yes)
-		(property "Reference" "C36"
+		(property "Reference" "C28"
 			(at 115.57 102.8762 0)
 			(effects
@@
 			(project "haldex_controller"
 				(path "/f9b060b2-b7a5-478e-9a0d-346ba4acb11f/ac628dfb-9786-4488-a934-d1527b457eba"
-					(reference "C36")
+					(reference "C28")
 					(unit 1)
 				)
@@
 		(dnp no)
 		(fields_autoplaced yes)
-		(property "Reference" "#PWR074"
+		(property "Reference" "#PWR084"
 			(at 163.83 132.08 0)
 			(effects
@@
 			(project "haldex_controller"
 				(path "/f9b060b2-b7a5-478e-9a0d-346ba4acb11f/ac628dfb-9786-4488-a934-d1527b457eba"
-					(reference "#PWR074")
+					(reference "#PWR084")
 					(unit 1)
 				)
@@
 		(dnp no)
 		(fields_autoplaced yes)
-		(property "Reference" "C37"
+		(property "Reference" "C27"
 			(at 48.26 88.9062 0)
 			(effects
@@
 			(project "haldex_controller"
 				(path "/f9b060b2-b7a5-478e-9a0d-346ba4acb11f/ac628dfb-9786-4488-a934-d1527b457eba"
-					(reference "C37")
+					(reference "C27")
 					(unit 1)
 				)
@@
 		(dnp no)
 		(fields_autoplaced yes)
-		(property "Reference" "#PWR098"
+		(property "Reference" "#PWR081"
 			(at 113.03 118.11 0)
 			(effects
@@
 			(project "haldex_controller"
 				(path "/f9b060b2-b7a5-478e-9a0d-346ba4acb11f/ac628dfb-9786-4488-a934-d1527b457eba"
-					(reference "#PWR098")
+					(reference "#PWR081")
 					(unit 1)
 				)
@@
 		(dnp no)
 		(fields_autoplaced yes)
-		(property "Reference" "TP6"
+		(property "Reference" "TP7"
 			(at 115.57 84.3279 0)
 			(effects
@@
 			(project "haldex_controller"
 				(path "/f9b060b2-b7a5-478e-9a0d-346ba4acb11f/ac628dfb-9786-4488-a934-d1527b457eba"
-					(reference "TP6")
+					(reference "TP7")
 					(unit 1)
 				)
@@
 		(dnp no)
 		(fields_autoplaced yes)
-		(property "Reference" "#PWR099"
+		(property "Reference" "#PWR078"
 			(at 45.72 107.95 0)
 			(effects
@@
 			(project "haldex_controller"
 				(path "/f9b060b2-b7a5-478e-9a0d-346ba4acb11f/ac628dfb-9786-4488-a934-d1527b457eba"
-					(reference "#PWR099")
+					(reference "#PWR078")
 					(unit 1)
 				)
@@
 		(dnp no)
 		(fields_autoplaced yes)
-		(property "Reference" "R43"
+		(property "Reference" "R40"
 			(at 97.79 82.5499 0)
 			(effects
@@
 			(project "haldex_controller"
 				(path "/f9b060b2-b7a5-478e-9a0d-346ba4acb11f/ac628dfb-9786-4488-a934-d1527b457eba"
-					(reference "R43")
+					(reference "R40")
 					(unit 1)
 				)
@@
 		(dnp no)
 		(fields_autoplaced yes)
-		(property "Reference" "TP2"
+		(property "Reference" "TP9"
 			(at 232.41 119.3799 90)
 			(effects
@@
 			(project "haldex_controller"
 				(path "/f9b060b2-b7a5-478e-9a0d-346ba4acb11f/ac628dfb-9786-4488-a934-d1527b457eba"
-					(reference "TP2")
+					(reference "TP9")
 					(unit 1)
 				)
@@
 		(dnp no)
 		(fields_autoplaced yes)
-		(property "Reference" "#PWR073"
+		(property "Reference" "#PWR083"
 			(at 154.94 87.63 0)
 			(effects
@@
 			(project "haldex_controller"
 				(path "/f9b060b2-b7a5-478e-9a0d-346ba4acb11f/ac628dfb-9786-4488-a934-d1527b457eba"
-					(reference "#PWR073")
+					(reference "#PWR083")
 					(unit 1)
 				)
@@
 		(dnp no)
 		(fields_autoplaced yes)
-		(property "Reference" "#PWR095"
+		(property "Reference" "#PWR079"
 			(at 66.04 68.58 0)
 			(effects
@@
 			(project "haldex_controller"
 				(path "/f9b060b2-b7a5-478e-9a0d-346ba4acb11f/ac628dfb-9786-4488-a934-d1527b457eba"
-					(reference "#PWR095")
+					(reference "#PWR079")
 					(unit 1)
 				)
@@
 		(dnp no)
 		(fields_autoplaced yes)
-		(property "Reference" "#FLG03"
+		(property "Reference" "#FLG010"
 			(at 77.47 62.865 0)
 			(effects
@@
 			(project "haldex_controller"
 				(path "/f9b060b2-b7a5-478e-9a0d-346ba4acb11f/ac628dfb-9786-4488-a934-d1527b457eba"
-					(reference "#FLG03")
+					(reference "#FLG010")
 					(unit 1)
 				)
@@
 		(dnp no)
 		(fields_autoplaced yes)
-		(property "Reference" "#PWR097"
+		(property "Reference" "#PWR080"
 			(at 102.87 118.11 0)
 			(effects
@@
 			(project "haldex_controller"
 				(path "/f9b060b2-b7a5-478e-9a0d-346ba4acb11f/ac628dfb-9786-4488-a934-d1527b457eba"
-					(reference "#PWR097")
+					(reference "#PWR080")
 					(unit 1)
 				)
@@
 		(dnp no)
 		(fields_autoplaced yes)
-		(property "Reference" "C26"
+		(property "Reference" "C30"
 			(at 157.48 74.9362 0)
 			(effects
@@
 			(project "haldex_controller"
 				(path "/f9b060b2-b7a5-478e-9a0d-346ba4acb11f/ac628dfb-9786-4488-a934-d1527b457eba"
-					(reference "C26")
+					(reference "C30")
 					(unit 1)
 				)
@@
 		(dnp no)
 		(fields_autoplaced yes)
-		(property "Reference" "FB5"
+		(property "Reference" "FB6"
 			(at 49.4919 63.5 90)
 			(effects
@@
 			(project "haldex_controller"
 				(path "/f9b060b2-b7a5-478e-9a0d-346ba4acb11f/ac628dfb-9786-4488-a934-d1527b457eba"
-					(reference "FB5")
+					(reference "FB6")
 					(unit 1)
 				)
@@
 		(dnp no)
 		(fields_autoplaced yes)
-		(property "Reference" "#FLG04"
+		(property "Reference" "#FLG011"
 			(at 132.08 86.995 0)
 			(effects
@@
 			(project "haldex_controller"
 				(path "/f9b060b2-b7a5-478e-9a0d-346ba4acb11f/ac628dfb-9786-4488-a934-d1527b457eba"
-					(reference "#FLG04")
-					(unit 1)
-				)
+					(reference "#FLG011")
+					(unit 1)
+				)
