File: wifi_nrf7002.kicad_sch (KiCad schematic)
At the start: 13 parts, among them IC2 TPS2553DBVT

Commit message: sch: fixing component footprints
Parts:
- FB6: footprint (none) -> Inductor_SMD:L_0805_2012Metric_Pad1.05x1.20mm_HandSolder
- IC2: footprint SOT95P280X145-6N -> TPS2553DBVT:SOT95P280X145-6N
- U7: footprint (none) -> ptr7002:ptr7002
Connections:
- net at U7.1 (NC), U7.18 (NC), U7.2 (NC)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: now also U7.33 (NC)
Changed lines of the file:
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@@
 			)
 		)
-		(property "Footprint" ""
+		(property "Footprint" "ptr7002:ptr7002"
 			(at 167.64 92.71 0)
 			(effects
@@
 			)
 		)
-		(property "Footprint" "SOT95P280X145-6N"
+		(property "Footprint" "TPS2553DBVT:SOT95P280X145-6N"
 			(at 87.63 190.17 0)
 			(effects
@@
 			)
 		)
-		(property "Footprint" ""
+		(property "Footprint" "Inductor_SMD:L_0805_2012Metric_Pad1.05x1.20mm_HandSolder"
 			(at 49.53 71.628 90)
 			(effects
