File: mcu.kicad_sch (KiCad schematic)
At the start: 57 parts, among them J2 BOOT0, J3 JTAG, J4 Debug, SW1 ~{RST}, SW2 Config, U2 STM32H573VITx, U3 PCA9557PW, U4 SST25VF080B-50-4x-S2Ax, U5 APS6404L-3SQR-SN, Y1 25MHz

Commit message: sch: fixing component footprints
Parts:
- SW1, SW2: footprint (none) -> TestPoint:TestPoint_Pad_D1.0mm

Commit message: sch: fix association with mounting holes and sw1/sw2
Parts:
- SW1: footprint TestPoint:TestPoint_Pad_D1.0mm -> Button_Switch_SMD:SW_Push_SPST_NO_Alps_SKRK
- SW2: footprint TestPoint:TestPoint_Pad_D1.0mm -> Button_Switch_SMD:SW_DIP_SPSTx04_Slide_Copal_CHS-04A_W5.08mm_P1.27mm_JPin

Commit message: working on component placement
Connections:
- net GND: now also R30.2, R31.2, R32.2, R33.2, R34.2, R35.2, R36.2, R37.2; no longer D10.1 (K), D11.1 (K), D12.1 (K), D5.1 (K), D6.1 (K), D7.1 (K), D8.1 (K), D9.1 (K)
- net LED0: now also D11.2 (A); no longer R36.1
- net LED1: now also D12.2 (A); no longer R37.1
- net LED_BODY_ERR: now also D7.2 (A); no longer R32.1
- net LED_BODY_RX: now also D6.2 (A); no longer R31.1
- net LED_BODY_TX: now also D5.2 (A); no longer R30.1
- net LED_HLDX_ERR: now also D10.2 (A); no longer R35.1
- net LED_HLDX_RX: now also D9.2 (A); no longer R34.1
- net LED_HLDX_TX: now also D8.2 (A); no longer R33.1
- new net: D5.1 (K), R30.1
- new net: D11.1 (K), R36.1
- new net: D7.1 (K), R32.1
- new net: D6.1 (K), R31.1
- new net: D9.1 (K), R34.1
- new net: D8.1 (K), R33.1
- new net: D12.1 (K), R37.1
- new net: D10.1 (K), R35.1
Other:
- moved on the sheet: D10, D11, D12, D5, D6, D7, D8, D9, R30, R31, R32, R33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

Commit message: brd: routing in progress
Parts:
- added C50: 100n, Capacitor_SMD:C_0603_1608Metric_Pad1.08x0.95mm_HandSolder, symbol Device:C_Small
- J2: footprint Connector_PinHeader_2.54mm:PinHeader_1x02_P2.54mm_Vertical -> Connector_PinHeader_1.27mm:PinHeader_1x02_P1.27mm_Vertical
- U4: footprint Package_SO:SOIC-8_5.275x5.275mm_P1.27mm -> Package_SO:SOIC-8_3.9x4.9mm_P1.27mm
Connections:
- net +3V3: now also C50.1
- net DIP_3: now also U2.62 (PD15); no longer U2.61 (PD14)
- net DIP_4: now also U2.61 (PD14); no longer U2.62 (PD15)
- net GND: now also D10.1 (K), D11.1 (K), D12.1 (K), D5.1 (K), D6.1 (K), D7.1 (K), D8.1 (K), D9.1 (K), C50.2; no longer R30.2, R31.2, R32.2, R33.2, R34.2, R35.2, R36.2, R37.2
- net HLDX_CAN_S: now also U2.2 (PE3); no longer U2.93 (PB7)
- net LED0: now also R36.1, U3.7 (IO1); no longer D11.2 (A), U3.13 (IO6)
- net LED1: now also R37.1, U3.6 (IO0); no longer D12.2 (A), U3.14 (IO7)
- net LED_BODY_ERR: now also R32.1; no longer D7.2 (A)
- net LED_BODY_RX: now also R31.1, U3.11 (IO4); no longer D6.2 (A), U3.7 (IO1)
- net LED_BODY_TX: now also R30.1, U3.13 (IO6); no longer D5.2 (A), U3.6 (IO0)
- net LED_HLDX_ERR: now also R35.1, U3.10 (IO3); no longer D10.2 (A), U3.12 (IO5)
- net LED_HLDX_RX: now also R34.1, U3.12 (IO5); no longer D9.2 (A), U3.11 (IO4)
- net LED_HLDX_TX: now also R33.1, U3.14 (IO7); no longer D8.2 (A), U3.10 (IO3)
- new net: D5.2 (A), R30.2
- new net: D11.2 (A), R36.2
- new net: D7.2 (A), R32.2
- new net: D6.2 (A), R31.2
- new net: D9.2 (A), R34.2
- new net: D8.2 (A), R33.2
- new net: D12.2 (A), R37.2
- new net: D10.2 (A), R35.2
Other:
- moved on the sheet: D10, D11, D12, D5, D6, D7, D8, D9, R30, R31, R32, R33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

Commit message: brd: layout complete
Parts:
- added C27: 100n, Capacitor_SMD:C_0603_1608Metric_Pad1.08x0.95mm_HandSolder, symbol Device:C_Small
Connections:
- net +3V3: now also C27.1
- net GND: now also C27.2
