File: grippyboi.kicad_pcb (KiCad board)
At the start: 4 copper layers, 68 x 100 mm, 204 parts, among them IC1 TPS62A02DRLR, IC3 LBEE5KL1YN-814, IC4 TLIN1027DRQ1, J1 GND, J10 12V in, J15 nRF7002 Ext, J2 BOOT0, J3 JTAG, J4 Debug, J5 USB, J6 MM8130-2600RA2, J7 Body 120R, J8 Hldx 120R, J9 ECU Connector, Q1 STR1550, Q2 BC807, Q3 Si7119DN, SW1 ~{RST}, SW2 Config, U1 LMR33630BDDA, U10 G3VM-61VY2, U11 G3VM-61VY2, U12 G3VM-61VY2, U13 G3VM-61VY2, U14 G3VM-61VY2, U15 G3VM-61VY2, U16 G3VM-61VY2, U17 G3VM-61VY2, U2 STM32H573VITx, U3 PCA9557PW, U4 SST25VF080B-50-4x-S2Ax, U5 APS6404L-3SQR-SN, U6 USBLC6-2SC6, U8 TJA1051T-3, U9 TJA1051T-3, X1 32.768kHz, Y1 25MHz

Commit message: brd: layer order marker added
Other:
- board text added: "1"
- board text added: "2"
- board text added: "3"
- board text added: "4"
Changed lines of the file:
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@@
 		(layer "Edge.Cuts")
 	)
+	(gr_text "1"
+		(at 97.282 76.073 90)
+		(layer "F.Cu")
+		(effects
+			(font
+				(size 1 1)
+				(thickness 0.1)
+			)
+			(justify left bottom)
+		)
+	)
+	(gr_text "2"
+		(at 97.282 75.057 90)
+		(layer "In1.Cu")
+		(effects
+			(font
+				(size 1 1)
+				(thickness 0.1)
+			)
+			(justify left bottom)
+		)
+	)
+	(gr_text "3"
+		(at 97.282 72.898 90)
+		(layer "In2.Cu")
+		(effects
+			(font
+				(size 1 1)
+				(thickness 0.1)
+			)
+			(justify left bottom mirror)
+		)
+	)
+	(gr_text "4"
+		(at 97.282 71.755 90)
+		(layer "B.Cu")
+		(effects
+			(font
+				(size 1 1)
+				(thickness 0.1)
+			)
+			(justify left bottom mirror)
+		)
+	)
 	(gr_text "Brake"
 		(at 103.290098 113.00797 0)
@@
 			)
 		)
+	)
+	(zone
+		(net 0)
+		(net_name "")
+		(layers "*.Mask" "F.Cu" "In1.Cu" "In2.Cu" "B.Cu")
+		(hatch edge 0.5)
+		(connect_pads
+			(clearance 0)
+		)
+		(min_thickness 0.25)
+		(filled_areas_thickness no)
+		(keepout
+			(tracks not_allowed)
+			(vias not_allowed)
+			(pads not_allowed)
+			(copperpour not_allowed)
+			(footprints not_allowed)
+		)
+		(fill
+			(thermal_gap 0.5)
+			(thermal_bridge_width 0.5)
+		)
+		(polygon
+			(pts
+				(xy 95.504 71.501) (xy 97.79 71.501) (xy 97.79 76.327) (xy 95.504 76.327)
+			)
+		)
